File: Eagle/ESP_DIN_V1.1.sch (EAGLE design)
At the start: 60 parts, among them IC1 TLP185, K1 HF46F/005-HS1, K2 44.62.9.006.0000, T1 BC817, T2 BC817, U1 ESP8266-12, U2 RXB6, U3 LM1117-3.3, X1 KF350-3.5-2P, X2 KF350-3.50-3P, X3 SMA-EDGE-UFLLONG, X4 KF301-5.08-2P, X5 KF301-5.08-2P, X6 KF301-5.08-3P, X8 KF301-5.08-2P

Commit message: readme + optocoupler fix
Changed lines of the file:
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@@
 <part name="R11" library="rcl" library_urn="urn:adsk.eagle:library:334" deviceset="R-EU_" device="R2010" package3d_urn="urn:adsk.eagle:package:23551/2" value="200K"/>
 <part name="D3" library="my-diode" deviceset="SL1*" device="" technology="M"/>
-<part name="GND15" library="supply1" library_urn="urn:adsk.eagle:library:371" deviceset="GND" device=""/>
 <part name="+3V13" library="supply1" library_urn="urn:adsk.eagle:library:371" deviceset="+3V3" device=""/>
 <part name="R13" library="rcl" library_urn="urn:adsk.eagle:library:334" deviceset="R-EU_" device="R0805" package3d_urn="urn:adsk.eagle:package:23553/2" value="10K"/>
@@
 <instance part="R11" gate="G$1" x="137.16" y="-15.24"/>
 <instance part="D3" gate="G$1" x="147.32" y="-17.78" rot="R90"/>
-<instance part="GND15" gate="1" x="170.18" y="-33.02"/>
 <instance part="+3V13" gate="G$1" x="177.8" y="0"/>
 <instance part="R13" gate="G$1" x="177.8" y="-25.4" rot="R90"/>
@@
 <segment>
 <pinref part="IC1" gate="G$1" pin="EMIT"/>
-<pinref part="GND15" gate="1" pin="GND"/>
-<wire x1="170.18" y1="-20.32" x2="170.18" y2="-30.48" width="0.1524" layer="91"/>
 <pinref part="R13" gate="G$1" pin="2"/>
 <wire x1="170.18" y1="-20.32" x2="177.8" y2="-20.32" width="0.1524" layer="91"/>
-<junction x="170.18" y="-20.32"/>
 <pinref part="C11" gate="G$1" pin="1"/>
 <wire x1="177.8" y1="-20.32" x2="193.04" y2="-20.32" width="0.1524" layer="91"/>

Commit message: IN & RF together
Parts:
- removed JP3: FTDI_CONN, my-connectors:FTDI_CONN
- removed X8: KF301-5.08-2P, my-connectors:KF301-5.08-2P
- added J1: (no value), SparkFun-Connectors:I2C_STANDARD_NO_SILK
- added X7: KF350-3.50-3P, my-connectors:KF350-3.50-3P
- C1: value 1000uF/16V -> 100n; device rcl:CPOL-EUTT5D10 -> rcl:C-EUC0805
- C12: value R463I24705001K -> 100uF/16V; device rcl:C-EU150-084X183 -> rcl:CPOL-EUE2-5
- C2, C5: value 100uF/16V -> 100n; device rcl:CPOL-EUE2-5 -> rcl:C-EUC0805
- C3, C7: value 100n -> R463I24705001K; device rcl:C-EUC0805 -> rcl:C-EU150-084X183
- C4: value 100n -> 1000uF/16V; device rcl:C-EUC0805 -> rcl:CPOL-EUTT5D10
- C6: value 100n -> 100uF/16V; device rcl:C-EUC0805 -> rcl:CPOL-EUE2-5
- C8: value R463I24705001K -> 100n; device rcl:C-EU150-084X183 -> rcl:C-EUC0805
- D1: value (none) -> S1B; device my-diode:KBP307 -> my-diode:S1B
- D2: value S1B -> (none); device my-diode:S1B -> my-diode:KBP307
- D3: value SL1M -> S1B; device my-diode:SL1M -> my-diode:S1B
- D5: value S1B -> SL1M; device my-diode:S1B -> my-diode:SL1M
- JP1: value (none) -> FTDI_CONN; device SparkFun-Connectors:I2C_STANDARD_NO_SILK -> my-connectors:FTDI_CONN
- R1: value S07K275 -> 820R; device varistor:S07K250 -> rcl:R-EU_R0805
- R10: value 820R -> 10K
- R11: value 200K -> 160R
- R12: value 4K7 -> 160R; device rcl:R-EU_R0805 -> rcl:R-EU_R2010
- R13: value 10K -> 200K; device rcl:R-EU_R0805 -> rcl:R-EU_R2010
- R14, R15: value 160R -> 4K7; device rcl:R-EU_R2010 -> rcl:R-EU_R0805
- R16: value 160R -> 10K; device rcl:R-EU_R2010 -> rcl:R-EU_R0805
- R2: value 10K -> 1K
- R4: value 10K -> S07K275; device rcl:R-EU_R0805 -> varistor:S07K250
- R7: value 1K -> 160R; device rcl:R-EU_R0805 -> rcl:R-EU_R2010
- R8: value 4K7 -> 1K
- R9: value 1K -> 10K
- U2: value RXB6 -> LM1117-3.3; device my-modules:RXB6 -> my-power:LM1117-3.3
- U3: value LM1117-3.3 -> RXB6; device my-power:LM1117-3.3 -> my-modules:RXB6
- X1: value KF350-3.5-2P -> KF301-5.08-3P; device my-connectors:KF350-3.5-2P -> my-connectors:KF301-5.08-3P
- X2: value KF350-3.50-3P -> KF301-5.08-2P; device my-connectors:KF350-3.50-3P -> my-connectors:KF301-5.08-2P
- X3: value SMA-EDGE-UFLLONG -> KF301-5.08-2P; device my-connectors:SMA-EDGE-UFLLONG -> my-connectors:KF301-5.08-2P
- X5: value KF301-5.08-2P -> KF350-3.5-2P; device my-connectors:KF301-5.08-2P -> my-connectors:KF350-3.5-2P
- X6: value KF301-5.08-3P -> SMA-EDGE-UFLLONG; device my-connectors:KF301-5.08-3P -> my-connectors:SMA-EDGE-UFLLONG
- renumbered D7 to D4, T1 to Q1, T2 to Q2
Connections:
- removed net GPIO15: R2.2, U1.GPIO15
- removed net N$1: LED1.A, U1.GPIO16
- new net INPUT: R13.1, X1-1.KL
- new net LED: LED1.A, R10.2, U1.GPIO15
- net +3V3: now also C2.1, C6.+, C8.1, J1.2, JP1.VCC, R14.2, R15.1, R9.2, U2.OUT, U3.VCC, X7-3.KL; no longer C2.+, C4.1, C7.1, JP1.2, JP3.VCC, R12.2, R4.2, R8.1, U2.VCC, U3.OUT, X2-3.KL
- net 1-WIRE: now also R15.2, X7-2.KL; no longer R8.2, X2-2.KL
- net ANT: now also U3.ANT, X6.ANT; no longer U2.ANT, X3.ANT
- net BUTTON: now also R9.1, X5-2.KL; no longer R5.1, X1-2.KL
- net CH: now also C1.1; no longer C6.1
- net DTR: now also JP1.DTR; no longer JP3.DTR
- net E: now also X1-2.KL, X1-3.KL; no longer X6-2.KL, X6-3.KL
- net GND: now also C12.-, C2.2, C4.-, C5.2, C6.-, C8.2, D2.-, J1.1, JP1.GND, R1.1, R16.1, X5-1.KL, X6.GND1, X6.GND2, X6.GND3, X6.GND4, X7-1.KL; no longer C1.-, C2.-, C3.2, C4.2, C5.-, C7.2, D1.-, JP1.1, JP3.GND, R13.1, R2.1, X1-1.KL, X2-1.KL, X3.GND1, X3.GND2, X3.GND3, X3.GND4
- net IN: now also C11.1, C12.+, IC1.EMIT, R16.2, U1.GPIO16; no longer R11.1, X6-1.KL
- net K1_POLE1: now also D1.A; no longer D2.A
- net K2_POLE1: now also D3.A; no longer D5.A
- net L: now also X2-2.KL; no longer X5-2.KL
- net L1_OUT: now also X3-1.KL; no longer X4-1.KL
- net L2_OUT: now also R11.2, X4-1.KL; no longer R16.2, X8-1.KL
- net N: now also C3.2, C7.2, X2-1.KL, X3-2.KL; no longer C12.2, C8.2, X4-2.KL, X5-1.KL
- net N$10: now also R5.1; no longer R3.1
- net N$11: now also C1.2, R3.1; no longer C6.2, R4.1
- net N$12: now also R7.2; no longer R14.2
- net N$13: now also C7.1, R12.1; no longer C8.1, R15.1
- net N$14: now also R4.1; no longer R1.1
- net N$15: now also R11.1, R12.2; no longer R15.2, R16.1
- net N$16: now also R2.1; no longer R7.1
- net N$2: now also R8.1; no longer R9.1
- net N$3: now also D2.AC1; no longer D1.AC1
- net N$4: now also D2.AC2; no longer D1.AC2
- net N$5: now also R1.2; no longer R10.2
- net N$6: now also D5.A; no longer D3.A
- net N$7: now also D5.C, R13.2; no longer D3.C, R11.2
- net N$8: now also R4.2; no longer R1.2
- net N$9: now also C3.1, R7.1; no longer C12.1, R14.1
- net N2_OUT: now also X4-2.KL; no longer X8-2.KL
- net RELAY1: now also R2.2; no longer R7.2
- net RELAY2: now also R8.2; no longer R9.2
- net RF: now also U3.DATA; no longer C11.1, C5.+, IC1.EMIT, R13.2, U2.DATA
- net RX: now also JP1.RXI; no longer JP3.RXI
- net SCL: now also J1.4, R14.1; no longer JP1.4, R12.1
- net SDA: now also J1.3; no longer JP1.3
- net TX: now also JP1.TXO; no longer JP3.TXO
- net VCC: now also C4.+, C5.1, D1.C, D2.+, D3.C, U2.IN; no longer C1.+, C3.1, D1.+, D2.C, D5.C, U3.IN
Other:
- note removed: "Do not solder if using RF receiver"
- moved on the sheet: C11, C3, C7, C8, D3, D5, LED1, R10, R11, R12, R13, R14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
